File: design/kicad/CPU.kicad_sch (KiCad schematic)
At the start: 8 parts, among them IC1 MC68010P10, Q2 5H8ET-10.000

Commit message: SolderDemon m68k r2.42: CPLD board, rebranding and silkscreen cleanup
Rename the KiCad project to solderdemon_m68k and move the glue logic
to two ATF1502AS CPLDs, with generator/routing scripts in design/tools.

Remove the upstream silkscreen badges (WEEE bin, OSHW certification
block, rosco_m68k logos, GitHub URL next to the expansion connector)
and bump the copyright to 2019-2026 via design/tools/strip_silk.py.
Other:
- company: The Really Old-School Company Limited -> SolderDemon
- title: ROSCO_M68K GENERAL PURPOSE MC68010 COMPUTER -> SolderDemon m68k Classic v2
Changed lines of the file:
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@@
   (paper "A4")
   (title_block
-    (title "ROSCO_M68K GENERAL PURPOSE MC68010 COMPUTER")
-    (date "2023-12-10")
-    (rev "2.13-DEV")
-    (company "The Really Old-School Company Limited")
+    (title "SolderDemon m68k Classic v2")
+    (date "2026-09-28")
+    (rev "2.42")
+    (company "SolderDemon")
     (comment 1 "OSHWA UK000006 (https://certification.oshwa.org/uk000006.html)")
     (comment 2 "See https://github.com/roscopeco/rosco_m68k/blob/master/LICENCE.hardware.txt")
     (comment 3 "Open Source Hardware licenced under CERN Open Hardware Licence")
     (comment 4 "Copyright 2019-2023 Ross Bamford and Contributors")
+    (comment 5 "SolderDemon modification 2026-09-28; based on rosco_m68k")
   )
   (junction (at 184.15 41.91) (diameter 0) (color 0 0 0 0)
@@
     (pin "2")
     (instances
-      (project "rosco_m68k"
+      (project "solderdemon_m68k"
         (path "/9031bb33-c6aa-4758-bf5c-3274ed3ebab7/00000000-0000-0000-0000-00005e53b4b8"
           (reference "R7") (unit 1)
@@
     (pin "2")
     (instances
-      (project "rosco_m68k"
+      (project "solderdemon_m68k"
         (path "/9031bb33-c6aa-4758-bf5c-3274ed3ebab7/00000000-0000-0000-0000-00005e53b4b8"
           (reference "R9") (unit 1)
@@
     (pin "2")
     (instances
-      (project "rosco_m68k"
+      (project "solderdemon_m68k"
         (path "/9031bb33-c6aa-4758-bf5c-3274ed3ebab7/00000000-0000-0000-0000-00005e53b4b8"
           (reference "R10") (unit 1)
@@
     (pin "1")
     (instances
-      (project "rosco_m68k"
+      (project "solderdemon_m68k"
         (path "/9031bb33-c6aa-4758-bf5c-3274ed3ebab7/00000000-0000-0000-0000-00005e53b4b8"
           (reference "#PWR01") (unit 1)
@@
     (pin "1")
     (instances
-      (project "rosco_m68k"
+      (project "solderdemon_m68k"
         (path "/9031bb33-c6aa-4758-bf5c-3274ed3ebab7/00000000-0000-0000-0000-00005e53b4b8"
           (reference "#PWR02") (unit 1)
@@
     (pin "1")
     (instances
-      (project "rosco_m68k"
+      (project "solderdemon_m68k"
         (path "/9031bb33-c6aa-4758-bf5c-3274ed3ebab7/00000000-0000-0000-0000-00005e53b4b8"
           (reference "#PWR03") (unit 1)
@@
     (pin "2")
     (instances
-      (project "rosco_m68k"
+      (project "solderdemon_m68k"
         (path "/9031bb33-c6aa-4758-bf5c-3274ed3ebab7/00000000-0000-0000-0000-00005e53b4b8"
           (reference "C7") (unit 1)
@@
     (pin "2")
     (instances
-      (project "rosco_m68k"
+      (project "solderdemon_m68k"
         (path "/9031bb33-c6aa-4758-bf5c-3274ed3ebab7/00000000-0000-0000-0000-00005e53b4b8"
           (reference "C8") (unit 1)
@@
     (pin "8")
     (instances
-      (project "rosco_m68k"
+      (project "solderdemon_m68k"
         (path "/9031bb33-c6aa-4758-bf5c-3274ed3ebab7/00000000-0000-0000-0000-00005e53b4b8"
           (reference "Q2") (unit 1)
@@
     (pin "2")
     (instances
-      (project "rosco_m68k"
+      (project "solderdemon_m68k"
         (path "/9031bb33-c6aa-4758-bf5c-3274ed3ebab7/00000000-0000-0000-0000-00005e53b4b8"
           (reference "R3") (unit 1)
@@
     (pin "53")
     (instances
-      (project "rosco_m68k"
+      (project "solderdemon_m68k"
         (path "/9031bb33-c6aa-4758-bf5c-3274ed3ebab7/00000000-0000-0000-0000-00005e53b4b8"
           (reference "IC1") (unit 1)
