File: design/kicad/DUART.kicad_sch (KiCad schematic)
At the start: 17 parts, among them IC4 XR68C681CJTR-F, J1 UART_A, J2 UART_B, J4 Conn_01x06, J7 Conn_01x01_Male, Q1 3.6864MHz

Commit message: SolderDemon m68k r2.42: CPLD board, rebranding and silkscreen cleanup
Rename the KiCad project to solderdemon_m68k and move the glue logic
to two ATF1502AS CPLDs, with generator/routing scripts in design/tools.

Remove the upstream silkscreen badges (WEEE bin, OSHW certification
block, rosco_m68k logos, GitHub URL next to the expansion connector)
and bump the copyright to 2019-2026 via design/tools/strip_silk.py.
Parts:
- removed J7: Conn_01x01_Male, Connector_PinHeader_2.54mm:PinHeader_1x01_P2.54mm_Vertical, symbol Connector:Conn_01x01_Pin
Other:
- company: The Really Old-School Company Limited -> SolderDemon
- title: ROSCO_M68K GENERAL PURPOSE MC68010 COMPUTER -> SolderDemon m68k Classic v2
Changed lines of the file:
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@@
   (paper "A4")
   (title_block
-    (title "ROSCO_M68K GENERAL PURPOSE MC68010 COMPUTER")
-    (date "2023-12-10")
-    (rev "2.13-DEV")
-    (company "The Really Old-School Company Limited")
+    (title "SolderDemon m68k Classic v2")
+    (date "2026-09-28")
+    (rev "2.42")
+    (company "SolderDemon")
     (comment 1 "OSHWA UK000006 (https://certification.oshwa.org/uk000006.html)")
     (comment 2 "See https://github.com/roscopeco/rosco_m68k/blob/master/LICENCE.hardware.txt")
     (comment 3 "Open Source Hardware licenced under CERN Open Hardware Licence")
     (comment 4 "Copyright 2019-2023 Ross Bamford and Contributors")
+    (comment 5 "SolderDemon modification 2026-09-28; based on rosco_m68k")
   )
   (junction (at 38.1 48.26) (diameter 0) (color 0 0 0 0)
@@
     )
   )
-  (global_label "SPICS2" (shape input) (at 96.52 143.51 180) (fields_autoplaced)
-    (effects (font (size 1.27 1.27)) (justify right))
-    (property "Intersheetrefs" "${INTERSHEET_REFS}" (at 0 0 0)
-      (effects (font (size 1.27 1.27)) hide)
-    )
-  )
   (global_label "SPIMOSI" (shape input) (at 95.25 161.29 180) (fields_autoplaced)
     (effects (font (size 1.27 1.27)) (justify right))
@@
     (pin "2")
     (instances
-      (project "rosco_m68k"
+      (project "solderdemon_m68k"
         (path "/9031bb33-c6aa-4758-bf5c-3274ed3ebab7/00000000-0000-0000-0000-000061622e90"
           (reference "Q1") (unit 1)
@@
     (pin "2")
     (instances
-      (project "rosco_m68k"
+      (project "solderdemon_m68k"
         (path "/9031bb33-c6aa-4758-bf5c-3274ed3ebab7/00000000-0000-0000-0000-000061622e90"
           (reference "C1") (unit 1)
@@
     (pin "2")
     (instances
-      (project "rosco_m68k"
+      (project "solderdemon_m68k"
         (path "/9031bb33-c6aa-4758-bf5c-3274ed3ebab7/00000000-0000-0000-0000-000061622e90"
           (reference "C2") (unit 1)
@@
     (pin "6")
     (instances
-      (project "rosco_m68k"
+      (project "solderdemon_m68k"
         (path "/9031bb33-c6aa-4758-bf5c-3274ed3ebab7/00000000-0000-0000-0000-000061622e90"
           (reference "J1") (unit 1)
@@
     (pin "6")
     (instances
-      (project "rosco_m68k"
+      (project "solderdemon_m68k"
         (path "/9031bb33-c6aa-4758-bf5c-3274ed3ebab7/00000000-0000-0000-0000-000061622e90"
           (reference "J2") (unit 1)
@@
     (pin "2")
     (instances
-      (project "rosco_m68k"
+      (project "solderdemon_m68k"
         (path "/9031bb33-c6aa-4758-bf5c-3274ed3ebab7/00000000-0000-0000-0000-000061622e90"
           (reference "C30") (unit 1)
@@
     (pin "2")
     (instances
-      (project "rosco_m68k"
+      (project "solderdemon_m68k"
         (path "/9031bb33-c6aa-4758-bf5c-3274ed3ebab7/00000000-0000-0000-0000-000061622e90"
           (reference "C28") (unit 1)
@@
     (pin "2")
     (instances
-      (project "rosco_m68k"
+      (project "solderdemon_m68k"
         (path "/9031bb33-c6aa-4758-bf5c-3274ed3ebab7/00000000-0000-0000-0000-000061622e90"
           (reference "C29") (unit 1)
@@
     (pin "9")
     (instances
-      (project "rosco_m68k"
+      (project "solderdemon_m68k"
         (path "/9031bb33-c6aa-4758-bf5c-3274ed3ebab7/00000000-0000-0000-0000-000061622e90"
           (reference "IC4") (unit 1)
@@
     (pin "2")
     (instances
-      (project "rosco_m68k"
+      (project "solderdemon_m68k"
         (path "/9031bb33-c6aa-4758-bf5c-3274ed3ebab7/00000000-0000-0000-0000-000061622e90"
           (reference "R1") (unit 1)
@@
     (pin "K")
     (instances
-      (project "rosco_m68k"
+      (project "solderdemon_m68k"
         (path "/9031bb33-c6aa-4758-bf5c-3274ed3ebab7/00000000-0000-0000-0000-000061622e90"
           (reference "LED1") (unit 1)
@@
     (pin "2")
     (instances
-      (project "rosco_m68k"
+      (project "solderdemon_m68k"
         (path "/9031bb33-c6aa-4758-bf5c-3274ed3ebab7/00000000-0000-0000-0000-000061622e90"
           (reference "R2") (unit 1)
@@
     (pin "K")
     (instances
-      (project "rosco_m68k"
+      (project "solderdemon_m68k"
         (path "/9031bb33-c6aa-4758-bf5c-3274ed3ebab7/00000000-0000-0000-0000-000061622e90"
           (reference "LED2") (unit 1)
@@
     (pin "1")
     (instances
-      (project "rosco_m68k"
+      (project "solderdemon_m68k"
         (path "/9031bb33-c6aa-4758-bf5c-3274ed3ebab7/00000000-0000-0000-0000-000061622e90"
           (reference "#PWR04") (unit 1)
@@
     (pin "6")
     (instances
-      (project "rosco_m68k"
+      (project "solderdemon_m68k"
         (path "/9031bb33-c6aa-4758-bf5c-3274ed3ebab7/00000000-0000-0000-0000-000061622e90"
           (reference "J4") (unit 1)
@@
     (pin "1")
     (instances
-      (project "rosco_m68k"
+      (project "solderdemon_m68k"
         (path "/9031bb33-c6aa-4758-bf5c-3274ed3ebab7/00000000-0000-0000-0000-000061622e90"
           (reference "#PWR0101") (unit 1)
@@
     (pin "1")
     (instances
-      (project "rosco_m68k"
+      (project "solderdemon_m68k"
         (path "/9031bb33-c6aa-4758-bf5c-3274ed3ebab7/00000000-0000-0000-0000-000061622e90"
           (reference "#PWR0102") (unit 1)
@@
     )
   )
-  (symbol (lib_id "Connector:Conn_01x01_Pin") (at 101.6 143.51 180) (unit 1)
-    (in_bom yes) (on_board yes) (dnp no)
-    (property "Reference" "J7" (at 99.06 139.7 0)
-      (effects (font (size 1.27 1.27)))
-    )
-    (property "Value" "Conn_01x01_Male" (at 98.8568 145.796 0)
-      (effects (font (size 1.27 1.27)))
-    )
-    (property "Footprint" "Connector_PinHeader_2.54mm:PinHeader_1x01_P2.54mm_Vertical" (at 101.6 143.51 0)
-      (effects (font (size 1.27 1.27)) hide)
-    )
-    (property "Datasheet" "~" (at 101.6 143.51 0)
-      (effects (font (size 1.27 1.27)) hide)
-    )
-    (pin "1")
-    (instances
-      (project "rosco_m68k"
-        (path "/9031bb33-c6aa-4758-bf5c-3274ed3ebab7/00000000-0000-0000-0000-000061622e90"
-          (reference "J7") (unit 1)
-        )
-      )
-    )
-  )
   (symbol (lib_id "Jumper:Jumper_2_Open") (at 254 143.51 0) (unit 1)
     (in_bom yes) (on_board yes) (dnp no)
@@
     (pin "2")
     (instances
-      (project "rosco_m68k"
+      (project "solderdemon_m68k"
         (path "/9031bb33-c6aa-4758-bf5c-3274ed3ebab7/00000000-0000-0000-0000-000061622e90"
           (reference "JP2") (unit 1)
@@
     (pin "2")
     (instances
-      (project "rosco_m68k"
+      (project "solderdemon_m68k"
         (path "/9031bb33-c6aa-4758-bf5c-3274ed3ebab7/00000000-0000-0000-0000-000061622e90"
           (reference "JP1") (unit 1)
