File: design/kicad/Expansion.kicad_sch (KiCad schematic)
At the start: 30 parts, among them IC1 MC68010P10, IC7 74LS148, J3 Conn_02x32_Odd_Even, J5 PWR, J6 Conn_01x05_Male, J8 Conn_01x02_Male

Commit message: SolderDemon m68k r2.42: CPLD board, rebranding and silkscreen cleanup
Rename the KiCad project to solderdemon_m68k and move the glue logic
to two ATF1502AS CPLDs, with generator/routing scripts in design/tools.

Remove the upstream silkscreen badges (WEEE bin, OSHW certification
block, rosco_m68k logos, GitHub URL next to the expansion connector)
and bump the copyright to 2019-2026 via design/tools/strip_silk.py.
Parts:
- removed J6: Conn_01x05_Male, Connector_PinHeader_2.54mm:PinHeader_1x05_P2.54mm_Vertical, symbol Connector:Conn_01x05_Pin
Other:
- company: The Really Old-School Company Limited -> SolderDemon
- title: ROSCO_M68K GENERAL PURPOSE MC68010 COMPUTER -> SolderDemon m68k Classic v2
