File: design/kicad/Reset.kicad_sch (KiCad schematic)
At the start: 12 parts, among them IC15 555N

Commit message: SolderDemon m68k r2.42: CPLD board, rebranding and silkscreen cleanup
Rename the KiCad project to solderdemon_m68k and move the glue logic
to two ATF1502AS CPLDs, with generator/routing scripts in design/tools.

Remove the upstream silkscreen badges (WEEE bin, OSHW certification
block, rosco_m68k logos, GitHub URL next to the expansion connector)
and bump the copyright to 2019-2026 via design/tools/strip_silk.py.
Other:
- company: The Really Old-School Company Limited -> SolderDemon
- title: ROSCO_M68K GENERAL PURPOSE MC68010 COMPUTER -> SolderDemon m68k Classic v2
Changed lines of the file:
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@@
   (paper "A4")
   (title_block
-    (title "ROSCO_M68K GENERAL PURPOSE MC68010 COMPUTER")
-    (date "2023-12-10")
-    (rev "2.13-DEV")
-    (company "The Really Old-School Company Limited")
+    (title "SolderDemon m68k Classic v2")
+    (date "2026-09-28")
+    (rev "2.42")
+    (company "SolderDemon")
     (comment 1 "OSHWA UK000006 (https://certification.oshwa.org/uk000006.html)")
     (comment 2 "See https://github.com/roscopeco/rosco_m68k/blob/master/LICENCE.hardware.txt")
     (comment 3 "Open Source Hardware licenced under CERN Open Hardware Licence")
     (comment 4 "Copyright 2019-2023 Ross Bamford and Contributors")
+    (comment 5 "SolderDemon modification 2026-09-28; based on rosco_m68k")
   )
   (junction (at 215.9 63.5) (diameter 0) (color 0 0 0 0)
@@
     (pin "8")
     (instances
-      (project "rosco_m68k"
+      (project "solderdemon_m68k"
         (path "/9031bb33-c6aa-4758-bf5c-3274ed3ebab7/00000000-0000-0000-0000-00006162e38e"
           (reference "IC15") (unit 1)
@@
     (pin "2")
     (instances
-      (project "rosco_m68k"
+      (project "solderdemon_m68k"
         (path "/9031bb33-c6aa-4758-bf5c-3274ed3ebab7/00000000-0000-0000-0000-00006162e38e"
           (reference "R27") (unit 1)
@@
     (pin "2")
     (instances
-      (project "rosco_m68k"
+      (project "solderdemon_m68k"
         (path "/9031bb33-c6aa-4758-bf5c-3274ed3ebab7/00000000-0000-0000-0000-00006162e38e"
           (reference "R28") (unit 1)
@@
     (pin "2")
     (instances
-      (project "rosco_m68k"
+      (project "solderdemon_m68k"
         (path "/9031bb33-c6aa-4758-bf5c-3274ed3ebab7/00000000-0000-0000-0000-00006162e38e"
           (reference "R14") (unit 1)
@@
     (pin "2")
     (instances
-      (project "rosco_m68k"
+      (project "solderdemon_m68k"
         (path "/9031bb33-c6aa-4758-bf5c-3274ed3ebab7/00000000-0000-0000-0000-00006162e38e"
           (reference "R31") (unit 1)
@@
     (pin "2")
     (instances
-      (project "rosco_m68k"
+      (project "solderdemon_m68k"
         (path "/9031bb33-c6aa-4758-bf5c-3274ed3ebab7/00000000-0000-0000-0000-00006162e38e"
           (reference "R32") (unit 1)
@@
     (pin "2")
     (instances
-      (project "rosco_m68k"
+      (project "solderdemon_m68k"
         (path "/9031bb33-c6aa-4758-bf5c-3274ed3ebab7/00000000-0000-0000-0000-00006162e38e"
           (reference "R13") (unit 1)
@@
     (pin "2")
     (instances
-      (project "rosco_m68k"
+      (project "solderdemon_m68k"
         (path "/9031bb33-c6aa-4758-bf5c-3274ed3ebab7/00000000-0000-0000-0000-00006162e38e"
           (reference "C13") (unit 1)
@@
     (pin "4")
     (instances
-      (project "rosco_m68k"
+      (project "solderdemon_m68k"
         (path "/9031bb33-c6aa-4758-bf5c-3274ed3ebab7/00000000-0000-0000-0000-00006162e38e"
           (reference "S1") (unit 1)
@@
     (pin "1")
     (instances
-      (project "rosco_m68k"
+      (project "solderdemon_m68k"
         (path "/9031bb33-c6aa-4758-bf5c-3274ed3ebab7/00000000-0000-0000-0000-00006162e38e"
           (reference "#SUPPLY01") (unit 1)
@@
     (pin "K")
     (instances
-      (project "rosco_m68k"
+      (project "solderdemon_m68k"
         (path "/9031bb33-c6aa-4758-bf5c-3274ed3ebab7/00000000-0000-0000-0000-00006162e38e"
           (reference "LED4") (unit 1)
@@
     (pin "K")
     (instances
-      (project "rosco_m68k"
+      (project "solderdemon_m68k"
         (path "/9031bb33-c6aa-4758-bf5c-3274ed3ebab7/00000000-0000-0000-0000-00006162e38e"
           (reference "LED3") (unit 1)
@@
     (pin "1")
     (instances
-      (project "rosco_m68k"
+      (project "solderdemon_m68k"
         (path "/9031bb33-c6aa-4758-bf5c-3274ed3ebab7/00000000-0000-0000-0000-00006162e38e"
           (reference "#SUPPLY02") (unit 1)
@@
     (pin "-")
     (instances
-      (project "rosco_m68k"
+      (project "solderdemon_m68k"
         (path "/9031bb33-c6aa-4758-bf5c-3274ed3ebab7/00000000-0000-0000-0000-00006162e38e"
           (reference "C11") (unit 1)
@@
     (pin "1")
     (instances
-      (project "rosco_m68k"
+      (project "solderdemon_m68k"
         (path "/9031bb33-c6aa-4758-bf5c-3274ed3ebab7/00000000-0000-0000-0000-00006162e38e"
           (reference "#PWR038") (unit 1)
@@
     (pin "1")
     (instances
-      (project "rosco_m68k"
+      (project "solderdemon_m68k"
         (path "/9031bb33-c6aa-4758-bf5c-3274ed3ebab7/00000000-0000-0000-0000-00006162e38e"
           (reference "#PWR036") (unit 1)
@@
     (pin "1")
     (instances
-      (project "rosco_m68k"
+      (project "solderdemon_m68k"
         (path "/9031bb33-c6aa-4758-bf5c-3274ed3ebab7/00000000-0000-0000-0000-00006162e38e"
           (reference "#PWR037") (unit 1)
@@
     (pin "1")
     (instances
-      (project "rosco_m68k"
+      (project "solderdemon_m68k"
         (path "/9031bb33-c6aa-4758-bf5c-3274ed3ebab7/00000000-0000-0000-0000-00006162e38e"
           (reference "#PWR039") (unit 1)
@@
     (pin "1")
     (instances
-      (project "rosco_m68k"
+      (project "solderdemon_m68k"
         (path "/9031bb33-c6aa-4758-bf5c-3274ed3ebab7/00000000-0000-0000-0000-00006162e38e"
           (reference "#PWR035") (unit 1)
@@
     (pin "1")
     (instances
-      (project "rosco_m68k"
+      (project "solderdemon_m68k"
         (path "/9031bb33-c6aa-4758-bf5c-3274ed3ebab7/00000000-0000-0000-0000-00006162e38e"
           (reference "#PWR034") (unit 1)
