File: design/kicad/solderdemon_m68k.kicad_pcb (KiCad board)
At the start: 4 copper layers, 160 x 100 mm, 86 parts, among them IC1 MC68010P10, IC15 555N, IC2 ATF1502AS-10JU44, IC3 ATF1502AS-10JU44, IC4 XR68C681CJTR-F, IC7 74LS148, J1 UART_A, J2 UART_B, J3 Conn_02x32_Odd_Even, J4 Conn_01x06, J5 PWR, J8 Conn_01x02_Male, J9 JTAG, Q1 3.6864MHz, Q2 5H8ET-10.000, U1 SST39SF040, U2 SST39SF040, U3 AS6C4008-55PCN, U4 AS6C4008-55PCN

Commit message: SolderDemon m68k r1: DUART in the CPLD column, own identity
Start SolderDemon's own revision numbering at r1. The board is 5 mm
longer (165 x 100 mm) so the DUART IC4 stands in one column with the
CPLDs IC3 and IC2: r1_layout.py stretches the r2.42 board along a cut
between the CPLDs and the CPU/RAM, bridging the crossing tracks, then
moves IC4 and reroutes it with KiCadRoutingTools.

The CPU decoupling C20/C12/C29/C31 stands in an even column in the
gap that opened, and the back carries the SolderDemon identity as on
the busboard (logo, name, "M68K Computer r1"). Silkscreen text moves
off the missing Futura font. trim_stubs.py cuts router overshoots
back to their junctions; cpld_route.py now spells '/' in net names
the way the board file does.

README: SolderDemon's m68k line built on rosco_m68k, r1 summary and
KiCad renders, photo of the assembled r2.42 board.
Parts:
- added LOGO1: SolderDemon_Logo, rosco_m68k:SolderDemon_Logo, B.Cu at (150.0, 73.1)
- moved C22 32.0 mm to (210.6, 124.0)
- moved C20 6.05 mm to (175.8, 59.0), turned to -90 degrees
- moved C29 5.59 mm to (175.8, 71.0)
- moved C12 5.36 mm to (175.8, 65.0)
- moved C31 5.27 mm to (175.8, 77.0)
- moved C1 5.00 mm to (189.1, 138.4)
- moved C10 5.00 mm to (184.5, 151.3)
- moved C11 5.00 mm to (227.7, 86.1)
- moved C13 5.00 mm to (227.7, 79.5)
- moved C14 5.00 mm to (215.2, 110.3)
- moved C16 5.00 mm to (229.3, 142.9)
- moved C18 5.00 mm to (215.2, 119.3)
- moved C19 5.00 mm to (215.2, 128.4)
- moved C2 5.00 mm to (207.2, 138.4)
- moved C21 5.00 mm to (220.9, 142.8)
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Routing:
- net D2: track 303.2 -> 219.0 mm
- net FC0: track 141.6 -> 187.3 mm, vias 8 -> 14
- net A1: track 334.7 -> 374.1 mm, vias 14 -> 16
- net FC2: track 174.1 -> 210.2 mm, vias 14 -> 19
- net A10: track 229.1 -> 265.0 mm, vias 3 -> 17
- net A2: track 337.7 -> 358.8 mm, vias 9 -> 13
- net A18: track 304.7 -> 325.8 mm, vias 8 -> 12
- net A19: track 299.5 -> 317.8 mm, vias 11 -> 17
- net A3: track 302.6 -> 320.6 mm, vias 16 -> 21
- net GND: track 100.2 -> 82.4 mm, vias 7 -> 11
- net D7: track 272.5 -> 256.3 mm, vias 5 -> 6
- net RW: track 265.0 -> 276.8 mm, vias 4 -> 8
- net RXDB: track 23.6 -> 34.8 mm, vias 1 -> 0
- net D4: track 327.6 -> 316.9 mm, vias 6 -> 8
- net RTSB: track 26.6 -> 36.8 mm, vias 0 -> 3
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Other:
- board size 160 x 100 mm -> 165 x 100 mm
- board text added: "DUART"
- board text added: "M68K Computer r1"
- board text added: "Revision r1"
- board text added: "SolderDemon"
- board text removed: "Revision 2.42"
- board text removed: "SolderDemon m68k"
- board text removed: "revision 2.42"
